File: pcb/choc/kongChoc.kicad_sch (KiCad schematic)
At the start: 124 parts, among them J1 BL_CONN, J3 USB_C_Receptacle_USB2.0, J4 Conn_01x08, SW1 SW_Push, SW10 SW_Push, SW11 SW_Push, SW12 SW_Push, SW13 SW_Push, SW14 SW_Push, SW15 SW_Push, SW16 SW_Push, SW17 SW_Push, SW18 SW_Push, SW2 SW_Push, SW20 SW_Push, SW21 SW_Push, SW23 SW_Push, SW24 SW_Push, SW25 SW_Push, SW26 SW_Push, SW29 SW_Push, SW3 SW_Push, SW30 SW_Push, SW31 SW_Push, SW32 SW_Push, SW33 SW_Push, SW34 SW_Push, SW37 SW_Push, SW38 SW_Push, SW39 SW_Push, SW4 SW_Push, SW41 SW_Push, SW42 SW_Push, SW43 SW_Push, SW44 SW_Push, SW45 SW_Push, SW46 SW_Push, SW47 SW_Push, SW48 SW_Push, SW49 SW_Push, SW5 SW_Push, SW50 SW_Push, SW51 SW_Push, SW52 SW_Push, SW53 SW_Push, SW54 SW_Push, SW55 SW_Push, SW6 SW_Push, SW7 SW_Push, SW8 SW_Push, SW9 SW_Push, U1 RP2040, U2 XC6206PxxxMR, U3 USBLC6-2SC6, U4 W25Q128JVS, Y1 Crystal_GND24_Small

Commit message: fix off-grid left 3u switch
Parts:
- C1: footprint weteor:USB-C-12-Pin-MidMount -> weteor:C_0402_HandSolder
Changed lines of the file:
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@@
     (stroke (width 0) (type default) (color 0 0 0 0))
   )
+  (wire (pts (xy 135.255 169.545) (xy 161.29 169.545))
+    (stroke (width 0) (type default) (color 0 0 0 0))
+  )
   (wire (pts (xy 38.1 259.715) (xy 48.26 259.715))
     (stroke (width 0) (type solid) (color 0 0 0 0))
@@
     (stroke (width 0) (type default) (color 0 0 0 0))
   )
-  (wire (pts (xy 161.29 151.765) (xy 135.255 151.765))
-    (stroke (width 0) (type default) (color 0 0 0 0))
-  )
   (wire (pts (xy 88.265 63.5) (xy 88.265 81.915))
     (stroke (width 0) (type default) (color 0 0 0 0))
@@
     (stroke (width 0) (type default) (color 0 0 0 0))
   )
-  (wire (pts (xy 161.29 169.545) (xy 135.255 169.545))
-    (stroke (width 0) (type default) (color 0 0 0 0))
-  )
   (wire (pts (xy 143.51 38.1) (xy 146.05 38.1))
     (stroke (width 0) (type default) (color 0 0 0 0))
@@
     (stroke (width 0) (type default) (color 0 0 0 0))
   )
+  (wire (pts (xy 135.255 151.765) (xy 161.29 151.765))
+    (stroke (width 0) (type default) (color 0 0 0 0))
+  )
   (wire (pts (xy 114.3 19.05) (xy 114.3 25.4))
     (stroke (width 0) (type default) (color 0 0 0 0))
@@
     (property "Reference" "C1" (id 0) (at 34.9313 180.7931 90))
     (property "Value" "27pF" (id 1) (at 34.9313 183.33 90))
-    (property "Footprint" "weteor:USB-C-12-Pin-MidMount" (id 2) (at 34.925 186.055 0)
+    (property "Footprint" "weteor:C_0402_HandSolder" (id 2) (at 34.925 186.055 0)
       (effects (font (size 1.27 1.27)) hide)
     )
@@
     )
     (path "/b4d27bb5-3f98-475b-96c8-5f0b8fac91a5"
-      (reference "C1") (unit 1) (value "27pF") (footprint "weteor:USB-C-12-Pin-MidMount")
+      (reference "C1") (unit 1) (value "27pF") (footprint "weteor:C_0402_HandSolder")
     )
     (path "/788e6fc6-d3b0-46c7-8256-9162d14568c1"
